File: uhlink.kicad_pcb (KiCad board)
At the start: 2 copper layers, 86 parts, among them J1 USB_C_Receptacle_USB2.0_16P, J10 TTL_CTRL, J11 TTL, J12 TTL_EXTRA, J13 BOOT0_SEL, J14 BOOT1_SEL, J15 MCU_DEBUG, J2 ARM_JTAG_SWD_20, J3 STDC14, J4 ARM_JTAG_SWD_10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

Commit message: feat: basic layout
Parts:
- J8, J9: footprint Connector_JST:JST_SH_SM03B-SRSS-TB_1x03-1MP_P1.00mm_Horizontal -> Connector_JST:JST_SH_BM03B-SRSS-TB_1x03-1MP_P1.00mm_Vertical
- moved J14 57.6 mm to (82.7, 70.5), turned to 0 degrees
- moved J13 52.4 mm to (86.2, 70.5), turned to 0 degrees
- moved J5 50.9 mm to (78.8, 41.0), turned to -90 degrees
- moved J15 45.8 mm to (90.3, 66.6)
- moved R12 44.8 mm to (85.8, 39.8), turned to 180 degrees
- moved R11 44.5 mm to (85.8, 38.2), turned to 180 degrees
- moved J2 44.4 mm to (116.6, 72.0), turned to -90 degrees
- moved JP1 39.3 mm to (97.2, 60.8), turned to 180 degrees
- moved Y1 34.0 mm to (98.8, 65.5), turned to 0 degrees
- moved R5 31.8 mm to (107.6, 67.3), turned to -90 degrees
- moved R7 31.8 mm to (111.6, 67.3), turned to -90 degrees
- moved U6 31.1 mm to (90.3, 52.8)
- moved C16 31.1 mm to (88.1, 52.8)
- moved C6 30.0 mm to (99.8, 62.4), turned to 180 degrees
- moved J9 29.7 mm to (109.7, 47.3), turned to 180 degrees
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Connections:
- U1 pad 31: unconnected-(U1-PA10-Pad31) -> /ARM20_I_JTDO_TRACESWO
- U1 pad 32: /HUB_USB1D- -> /HUB_USB4D-
- U1 pad 33: /HUB_USB1D+ -> /HUB_USB4D+
- U5 pad 3: /HUB_USB2D+ -> /HUB_USB1D+
- U5 pad 4: /HUB_USB2D- -> /HUB_USB1D-
- U6 pad 1: /ESD_USBCD- -> /ESD_USBAD-
- U6 pad 3: /ESD_USBCD+ -> /ESD_USBAD+
- U6 pad 4: /HUB_USB4D+ -> /HUB_USB3D+
- U6 pad 6: /HUB_USB4D- -> /HUB_USB3D-
- U7 pad 1: /ESD_USBAD- -> /ESD_USBCD-
- U7 pad 3: /ESD_USBAD+ -> /ESD_USBCD+
- U7 pad 4: /HUB_USB3D+ -> /HUB_USB2D+
- U7 pad 6: /HUB_USB3D- -> /HUB_USB2D-
Routing:
- net /TTL_VIO: track 0.00 -> 44.7 mm, vias 0 -> 2
- net /TTL_TXD: track 0.00 -> 44.0 mm, vias 0 -> 3
- net /MCU_I_JTCK_SWCLK: track 0.00 -> 43.3 mm, vias 0 -> 5
- net /MCU_I_JTMS_SWDIO: track 0.00 -> 39.5 mm, vias 0 -> 5
- net /TTL_RXD: track 0.00 -> 39.1 mm, vias 0 -> 3
- net /ARM20_I_JTDO_TRACESWO: track 0.00 -> 34.3 mm, vias 0 -> 3
- net /MCU_I_JTDI: track 0.00 -> 31.7 mm, vias 0 -> 3
- net /MCU_I_nRESET: track 0.00 -> 30.3 mm, vias 0 -> 3
- net VBUS: track 0.00 -> 21.7 mm, vias 0 -> 3
- net /TTL_RXS_GPIO1: track 0.00 -> 20.8 mm, vias 0 -> 2
- net /HUB_USB2D+: track 0.00 -> 20.8 mm
- net /MCU_JTMS_SWDIO: track 0.00 -> 20.7 mm
- net /HUB_USB2D-: track 0.00 -> 20.5 mm
- net /TTL_~{RESET}: track 0.00 -> 20.4 mm, vias 0 -> 1
- net /MCU_JTCK_SWCLK: track 0.00 -> 19.3 mm
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Other:
- copper layers 2 -> 4
